File: canfuel/canfuel.kicad_sch (KiCad schematic)
At the start: 24 parts, among them J1 Micro-Fit 43045-0400, J2 Micro-Fit 43045-0400, J3 ICSP, U1 PIC18F25K80, U2 MCP2562-E/P, Y1 16MHz

Commit message: D1 is red: the parts were tested before fitting
The two LEDs actually going on the board were checked on a multimeter's diode
range, both reading Vf around 1.8 V, and the choice landed on red for D1 rather
than green. Yellow for D2 is unchanged.

Changed at the source and propagated, rather than in prose: the schematic's
Value field for D1, then canfuel-bom.csv regenerated with the kicad-cli command
in plan 7. Exactly one line of the BOM moved and the format did not drift,
which is the point of regenerating rather than editing it. The parts table in
plan 2 and the reasoning here follow.

One derived number moved with it. The LED paragraph costed the range at Vf = 2 V
and Vf = 3.2 V, giving 2.3 mA and 1.1 mA. Red at the measured 1.8 V draws about
3.2 mA through the same 1 k, so the span is now stated as 3.2 mA down to 1.1 mA.
Still an order of magnitude under the 25 mA the port pin allows, so the
conclusion is untouched: colour is free and only brightness changes.

Nothing here reaches the PCB -- LED colour does not touch copper, and the three
boards already made are unaffected. check-netlist.py and check-placement.py both
still pass against the edited schematic.

Co-Authored-By: Claude Opus 5 <noreply@anthropic.com>
Claude-Session: https://claude.ai/code/session_01NSh4X115wJ5EQHBww5YVKm
Parts:
- D1: value green -> red
Changed lines of the file:
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@@
 		(property
 			"Value"
-			"green"
+			"red"
 			(at 261.62 233.68 0)
 			(show_name no)
