File: canfuel/canfuel.kicad_pcb (KiCad board)
At the start: 2 copper layers, 55 x 45 mm, 28 parts, among them J1 Micro-Fit 43045-0400, J2 Micro-Fit 43045-0400, J3 ICSP, U1 PIC18F25K80, U2 MCP2562-E/P, Y1 16MHz

Commit message: D1 is red in the board too, and fab/ deliberately still says green
The schematic and the board each carry their own Value field. kicad-cli takes
the BOM from one and the CPL from the other, so when D1 was changed to red in
the schematic alone, fab/canfuel-bom.csv said red and fab/canfuel-cpl.csv said
green and nothing complained. Neither ERC, DRC, check-netlist.py nor
check-placement.py reads Value; only import-footprints.py writes it, and that
is the step that was skipped. What found it was render-solder-check.py printing
the board's copy at the head of D1's table.

fab/ is left alone on purpose. It is the record of what was sent to the
manufacturer and the boards on the bench were made from exactly those files;
regenerating it to tidy up a colour would throw that away to fix something no
fab process reads. The two figures in canfuel/docs/ are generated now, so they
say red.

render-assembly.py stops hard-coding either the colour or the LED's resistor
and derives both -- the Value field the BOM comes from, and whatever else sits
on the anode net. The output is byte-identical to what it hard-coded, which is
the check that the derivation is the same answer rather than a new one.

check-netlist.py, check-placement.py and DRC all clean afterwards.

Co-Authored-By: Claude Opus 5 <noreply@anthropic.com>
Claude-Session: https://claude.ai/code/session_01MeNVAM1Z8QhuKcJykYAbrV
Parts:
- D1: value green -> red
Changed lines of the file:
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@@
 			)
 		)
-		(property "Value" "green"
+		(property "Value" "red"
 			(at 1.27 2.96 0)
 			(layer "F.Fab")
